File: schematic/macr0.sch (KiCad schematic (older format))
At the start: 25 parts, among them J1 USB_C_Receptacle_USB2.0, J2 AVR-ISP-6, U1 ATmega32U4-AU, U2 CAT4104, Y1 16MHz

Commit message: Finished schametic.  Working on PCB layout.
Parts:
- removed J1: USB_C_Receptacle_USB2.0, symbol Connector:USB_C_Receptacle_USB2.0
- added J1: USB_C_Receptacle, Connector_USB:USB_C_Receptacle_Amphenol_12401548E4-2A, symbol Connector:USB_C_Receptacle
- C1, C2, C3, C4: footprint (none) -> Capacitor_SMD:C_1206_3216Metric_Pad1.42x1.75mm_HandSolder
- D1, D2, D3, D4: footprint (none) -> Diode_SMD:D_SOD-123
- J2: footprint (none) -> Connector_IDC:IDC-Header_2x03_P2.54mm_Vertical
- R1, R2, R3, R4, R5, R6: footprint (none) -> Resistor_SMD:R_1206_3216Metric_Pad1.42x1.75mm_HandSolder
- R7: value R -> 6k; footprint (none) -> Resistor_SMD:R_1206_3216Metric_Pad1.42x1.75mm_HandSolder
- S0: footprint (none) -> Button_Switch_SMD:SW_Push_1P1T_NO_6x6mm_H9.5mm
- S1, S2, S3, S4: footprint (none) -> macr0:Gateron_LED_1.00u_Plate
- U2: footprint (none) -> macr0:CAT4101
- Y1: footprint (none) -> Crystal:Crystal_SMD_HC49-SD_HandSoldering
Connections:
- net +5V: now also J1.A4 (VBUS), J1.A9 (VBUS), J1.B4 (VBUS), J1.B9 (VBUS)
- net GND: now also J1.A1 (GND), J1.A12 (GND), J1.B1 (GND), J1.B12 (GND)
- net at R3.2: now also J1.A5 (CC1)
- net at R6.2: now also J1.A6 (D+), J1.B6 (D+)
- net at R5.2: now also J1.A7 (D-), J1.B7 (D-)
- net at R4.2: now also J1.B5 (CC2)
- no-connect marks 23 -> 31
Other:
- moved on the sheet: C4, R3, R4, R5, R6

Commit message: First prototype pcb for fab.
Parts:
- J2: footprint Connector_IDC:IDC-Header_2x03_P2.54mm_Vertical -> Connector_PinHeader_2.54mm:PinHeader_2x03_P2.54mm_Vertical
Other:
- note added: "20200726"
- note added: "2x2 Button Matrix"
- note added: "ATmega32U4 AVR Microcontroller"
- note added: "AVR In-System Programmer"
- note added: "CAT4104 Constand Current LED Driver"
- note added: "USB-C Receptacle\nConfigured to identify as USB 2.0 Device"
- note added: "macr0 - USB HID 2x2 Button Matrix with LED Illumination"
- note removed: "20200720"
- note removed: "macr0"
- moved on the sheet: C1, C2, C3, C4, J1, J2, R1, R2, R3, R4, R5, R6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
