File: hardware/macr0.kicad_pcb (KiCad board)
At the start: 2 copper layers, 43.2 x 43.2 mm, 26 parts, among them J1 USB-C, J2 AVR-ISP-6, U1 ATmega32U4-AU, U2 CAT4104, Y1 16MHz

Commit message: Silkscreen correction and improvements.
Parts:
- C2: value 22uF -> 22pF
- S0: value BRIGHTNESS -> DIMMER
Other:
- board text added: "!RST"
- board text added: "+5V"
- board text added: "GND"
- board text added: "MISO"
- board text added: "MOSI"
- board text added: "SCK"
Changed lines of the file:
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@@
   (general
     (thickness 1.6)
-    (drawings 5)
+    (drawings 11)
     (tracks 377)
     (zones 0)
@@
       (effects (font (size 1 1) (thickness 0.15)) (justify mirror))
     )
-    (fp_text value 22uF (at 1.3065 1.778) (layer B.SilkS)
+    (fp_text value 22pF (at 1.3065 1.778) (layer B.SilkS)
       (effects (font (size 1 1) (thickness 0.15)) (justify mirror))
     )
@@
       (effects (font (size 1 1) (thickness 0.15)) (justify mirror))
     )
-    (fp_text value 1uF (at 3.2655 0 180) (layer B.SilkS)
+    (fp_text value 1uF (at 3.0115 0 180) (layer B.SilkS)
       (effects (font (size 1 1) (thickness 0.15)) (justify mirror))
     )
@@
     )
     (fp_text value 1N4148 (at 0 1.905) (layer B.SilkS)
-      (effects (font (size 1 1) (thickness 0.15)) (justify mirror))
+      (effects (font (size 0.75 0.75) (thickness 0.15)) (justify mirror))
     )
     (fp_line (start -2.25 1) (end 1.65 1) (layer B.SilkS) (width 0.12))
@@
       (effects (font (size 1 1) (thickness 0.15)) (justify mirror))
     )
-    (fp_text value 1N4148 (at 1.397 1.905) (layer B.SilkS)
-      (effects (font (size 1 1) (thickness 0.15)) (justify mirror))
+    (fp_text value 1N4148 (at 1.651 1.905) (layer B.SilkS)
+      (effects (font (size 0.75 0.75) (thickness 0.15)) (justify mirror))
     )
     (fp_text user %R (at 0 2) (layer B.Fab)
@@
       (effects (font (size 1 1) (thickness 0.15)) (justify mirror))
     )
-    (fp_text value 1N4148 (at 1.778 -1.905) (layer B.SilkS)
-      (effects (font (size 1 1) (thickness 0.15)) (justify mirror))
+    (fp_text value 1N4148 (at 2.032 -1.651) (layer B.SilkS)
+      (effects (font (size 0.75 0.75) (thickness 0.15)) (justify mirror))
     )
     (fp_text user %R (at 0 2) (layer B.Fab)
@@
       (effects (font (size 1 1) (thickness 0.15)) (justify mirror))
     )
-    (fp_text value 1N4148 (at 0 1.778) (layer B.SilkS)
-      (effects (font (size 1 1) (thickness 0.15)) (justify mirror))
+    (fp_text value 1N4148 (at -0.508 1.778) (layer B.SilkS)
+      (effects (font (size 0.75 0.75) (thickness 0.15)) (justify mirror))
     )
     (fp_line (start -2.25 1) (end 1.65 1) (layer B.SilkS) (width 0.12))
@@
       (effects (font (size 1 1) (thickness 0.15)) (justify mirror))
     )
-    (fp_text value 10k (at -3.3385 -1.27 180) (layer B.SilkS)
+    (fp_text value 10k (at 1.4875 -2.54 180) (layer B.SilkS)
       (effects (font (size 1 1) (thickness 0.15)) (justify mirror))
     )
@@
       (effects (font (size 1 1) (thickness 0.15)) (justify mirror))
     )
-    (fp_text value 6k (at 0.0365 -1.778) (layer B.SilkS)
+    (fp_text value 6k (at 1.3065 -1.778) (layer B.SilkS)
       (effects (font (size 1 1) (thickness 0.15)) (justify mirror))
     )
@@
       (effects (font (size 1 1) (thickness 0.15)) (justify mirror))
     )
-    (fp_text value BRIGHTNESS (at -5.588 -0.254 180) (layer B.SilkS)
+    (fp_text value DIMMER (at -5.588 -0.254 180) (layer B.SilkS)
       (effects (font (size 1 1) (thickness 0.15)) (justify mirror))
     )
@@
     (tags "QFP 0.8")
     (attr smd)
-    (fp_text reference U1 (at 0 7.45 45) (layer B.SilkS)
+    (fp_text reference U1 (at 0 7.45 45) (layer B.SilkS) hide
       (effects (font (size 1 1) (thickness 0.15)) (justify mirror))
     )
@@
       (effects (font (size 1 1) (thickness 0.15)) (justify mirror))
     )
-    (fp_text value CAT4104 (at 0.508 -5.08 180) (layer B.SilkS)
+    (fp_text value CAT4104 (at 0 -5.08 180) (layer B.SilkS)
       (effects (font (size 1 1) (thickness 0.15)) (justify mirror))
     )
@@
     )
   )
+  (gr_text !RST (at 140.208 116.586 90) (layer B.SilkS)
+    (effects (font (size 0.5 0.5) (thickness 0.125)) (justify mirror))
+  )
+  (gr_text SCK (at 140.208 114.046 90) (layer B.SilkS)
+    (effects (font (size 0.5 0.5) (thickness 0.125)) (justify mirror))
+  )
+  (gr_text MISO (at 140.208 111.506 90) (layer B.SilkS)
+    (effects (font (size 0.5 0.5) (thickness 0.125)) (justify mirror))
+  )
+  (gr_text MOSI (at 134.112 114.046 90) (layer B.SilkS)
+    (effects (font (size 0.5 0.5) (thickness 0.125)) (justify mirror))
+  )
+  (gr_text +5V (at 134.112 111.252 90) (layer B.SilkS)
+    (effects (font (size 0.5 0.5) (thickness 0.125)) (justify mirror))
+  )
+  (gr_text GND (at 134.112 116.586 90) (layer B.SilkS)
+    (effects (font (size 0.5 0.5) (thickness 0.125)) (justify mirror))
+  )
   (gr_text clewsy.pro (at 127 117.348) (layer B.SilkS)

Commit message: I'm so bad at this, I can't even spell my name correctly.
Other:
- board text added: "clews.pro"
- board text removed: "clewsy.pro"
Changed lines of the file:
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@@
     (effects (font (size 0.5 0.5) (thickness 0.125)) (justify mirror))
   )
-  (gr_text clewsy.pro (at 127 117.348) (layer B.SilkS)
+  (gr_text clews.pro (at 127 117.348) (layer B.SilkS)
     (effects (font (size 0.75 0.75) (thickness 0.125)) (justify mirror))
   )

Commit message: Working on hardware rev2.
Parts:
- removed D1, D2, D3, D4: 1N4148, Diode_SMD:D_SOD-123
- removed R2: 10k, Resistor_SMD:R_1206_3216Metric_Pad1.42x1.75mm_HandSolder
- removed R7: 6k, Resistor_SMD:R_1206_3216Metric_Pad1.42x1.75mm_HandSolder
- removed U2: CAT4104, macr0:CAT4101
- added G***: LOGO, macr0:osha_logo_8mm, B.Cu at (-5.08, 19.3)
- added Q1: PNP, Package_TO_SOT_SMD:SOT-223-3_TabPin2, B.Cu at (29.5, -8.13)
- added R05: 22, Resistor_SMD:R_1206_3216Metric_Pad1.42x1.75mm_HandSolder, B.Cu at (8.13, -6.99)
- added R07: 50, Resistor_SMD:R_1206_3216Metric_Pad1.42x1.75mm_HandSolder, B.Cu at (30.5, 3.05)
- added R08: 50, Resistor_SMD:R_1206_3216Metric_Pad1.42x1.75mm_HandSolder, B.Cu at (30.5, 0.00)
- added R09: 50, Resistor_SMD:R_1206_3216Metric_Pad1.42x1.75mm_HandSolder, B.Cu at (30.5, 6.10)
- added R10: 50, Resistor_SMD:R_1206_3216Metric_Pad1.42x1.75mm_HandSolder, B.Cu at (30.5, 9.14)
- J1: value USB-C -> usb-c
- R6: value 22 -> 7k5
- U1: value ATmega32U4-AU -> ATmega32U4
- Y1: footprint Crystal:Crystal_SMD_HC49-SD_HandSoldering -> Crystal:Crystal_SMD_HC49-SD
- moved G*** 177.5 mm to (-4.57, -11.2)
- moved C4 166.5 mm to (12.1, -6.99), turned to 90 degrees
- moved R02 165.6 mm to (5.08, -14.0), turned to 270 degrees
- moved R01 165.1 mm to (6.35, 21.0), turned to 90 degrees
- moved R03 162.8 mm to (19.1, -14.0), turned to 90 degrees
- moved C2 160.9 mm to (0.00, 2.54)
- moved J1 158.7 mm to (9.09, -11.6)
- moved U1 157.7 mm to (12.1, 4.45), turned to 135 degrees
- moved Y1 157.2 mm to (-5.71, 4.45), turned to 90 degrees
- moved S1 155.1 mm to (0.00, 0.00), turned to 180 degrees
- moved S2 155.1 mm to (19.1, 0.00), turned to 180 degrees
- moved S3 155.1 mm to (0.00, 19.1), turned to 180 degrees
- moved S4 155.1 mm to (19.1, 19.1), turned to 180 degrees
- moved J2 155.0 mm to (10.8, 23.5), turned to 0 degrees
- moved C3 153.7 mm to (22.9, 4.45), turned to 90 degrees
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- renumbered R1 to R01, R3 to R02, R4 to R03, R5 to R04
Connections:
- R6 pad 1: D+ -> Net-(Q1-Pad1)
- R6 pad 2: Net-(J1-PadA6) -> LED_PWM
- S1 pad 1: Net-(D1-Pad2) -> KEY1
- S1 pad 2: COL1 -> Net-(S1-Pad2)
- S1 pad 4: Net-(S1-Pad4) -> Net-(S1-Pad2)
- S2 pad 1: Net-(D2-Pad2) -> KEY2
- S2 pad 2: COL2 -> GND
- S2 pad 3: Net-(S1-Pad4) -> LED2
- S2 pad 4: +5V -> GND
- S3 pad 1: Net-(D3-Pad2) -> KEY3
- S3 pad 2: COL1 -> Net-(S1-Pad2)
- S3 pad 3: LED2 -> LED3
- S3 pad 4: Net-(S3-Pad4) -> Net-(S1-Pad2)
- S4 pad 1: Net-(D4-Pad2) -> KEY4
- S4 pad 2: COL2 -> GND
- S4 pad 3: Net-(S3-Pad4) -> LED4
- S4 pad 4: +5V -> GND
- U1 pad 18: ROW1 -> KEY1
- U1 pad 19: ROW2 -> KEY2
- U1 pad 20: COL1 -> KEY3
- U1 pad 21: COL2 -> KEY4
Routing:
- net +5V: track 108.5 -> 0.00 mm, vias 3 -> 0
- net ROW1: track 52.3 -> 0.00 mm
- net Net-(S0-Pad1): track 49.9 -> 0.00 mm
- net GND: track 49.4 -> 0.00 mm, vias 11 -> 0
- net COL2: track 39.5 -> 0.00 mm, vias 1 -> 0
- net LED1: track 38.5 -> 0.00 mm, vias 1 -> 0
- net COL1: track 37.5 -> 0.00 mm
- net ROW2: track 35.9 -> 0.00 mm, vias 3 -> 0
- net D+: track 32.2 -> 0.00 mm, vias 2 -> 0
- net D-: track 31.7 -> 0.00 mm
- net LED2: track 30.7 -> 0.00 mm
- net !RESET: track 30.5 -> 0.00 mm
- net MISO: track 26.6 -> 0.00 mm
- net Net-(S1-Pad4): track 23.9 -> 0.00 mm
- net Net-(S3-Pad4): track 22.4 -> 0.00 mm
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- removed copper zone on B.Cu, net GND
- removed copper zone on F.Cu, net GND
Other:
- board size 43.2 x 43.2 mm -> 44.5 x 44.5 mm

Commit message: Working on hardware rev2.
Parts:
- J2: value AVR-ISP-6 -> AVR-ISP
- moved C2 4.06 mm to (0.00, 6.60)
- moved C1 3.81 mm to (0.00, 2.54)
- moved C4 0.67 mm to (12.1, -7.66)
- turned Y1 to 270 degrees
Connections:
- S1 pad 1: KEY1 -> GND
- S1 pad 2: Net-(S1-Pad2) -> KEY1
- S1 pad 3: LED1 -> GND
- S1 pad 4: Net-(S1-Pad2) -> LED1
- S2 pad 1: KEY2 -> GND
- S2 pad 2: GND -> KEY2
- S2 pad 3: LED2 -> GND
- S2 pad 4: GND -> LED2
- S3 pad 1: KEY3 -> GND
- S3 pad 2: Net-(S1-Pad2) -> KEY3
- S3 pad 3: LED3 -> GND
- S3 pad 4: Net-(S1-Pad2) -> LED3
- S4 pad 1: KEY4 -> GND
- S4 pad 2: GND -> KEY4
- S4 pad 3: LED4 -> GND
- S4 pad 4: GND -> LED4
Routing:
- net +5V: track 0.00 -> 163.0 mm, vias 0 -> 3
- net LED3: track 0.00 -> 45.1 mm
- net GND: track 0.00 -> 35.5 mm, vias 0 -> 5
- net LED1: track 0.00 -> 33.4 mm
- net KEY4: track 0.00 -> 25.0 mm, vias 0 -> 1
- net Net-(C1-Pad1): track 0.00 -> 23.2 mm
- net KEY2: track 0.00 -> 22.6 mm, vias 0 -> 1
- net Net-(Q1-Pad2): track 0.00 -> 21.9 mm
- net Net-(S0-Pad1): track 0.00 -> 21.7 mm
- net LED_PWM: track 0.00 -> 21.1 mm, vias 0 -> 2
- net Net-(C2-Pad1): track 0.00 -> 18.4 mm
- net D+: track 0.00 -> 17.1 mm
- net KEY1: track 0.00 -> 16.6 mm
- net D-: track 0.00 -> 16.5 mm
- net Net-(J1-PadS1): track 0.00 -> 15.4 mm
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- added copper zone on B.Cu, net GND
- added copper zone on F.Cu, net GND
